File: Schematic_PCB/RevoxESP32Light/RevoxESP32Light.kicad_sch (KiCad schematic)
At the start: 27 parts, among them J1 SerialLink, J2 Conn_01x04, J3 Conn_01x10, J4 Conn_01x05, J5 Conn_01x04, J6 Conn_01x03, Q1 BC550, Q2 2N2222, Q3 BC550, U1 esp32-wemos-d1-mini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

Commit message: N.V.
Parts:
- removed D1, D2, D3: LED, LED_THT:LED_D3.0mm_Horizontal_O1.27mm_Z2.0mm_IRBlack, symbol Device:LED
- removed Q1, Q3: BC550, Package_TO_SOT_THT:TO-92_Inline, symbol Transistor_BJT:BC550
- removed Q2: 2N2222, Package_TO_SOT_THT:TO-92_Inline, symbol Transistor_BJT:2N3904
- removed R1, R11, R3: 4,7k, Resistor_THT:R_Axial_DIN0309_L9.0mm_D3.2mm_P12.70mm_Horizontal, symbol Device:R
- removed R10, R4, R5: 22k, Resistor_THT:R_Axial_DIN0309_L9.0mm_D3.2mm_P12.70mm_Horizontal, symbol Device:R
- removed R2, R7, R9: 180, Resistor_THT:R_Axial_DIN0309_L9.0mm_D3.2mm_P12.70mm_Horizontal, symbol Device:R
Connections:
- net ~{EN1}: no longer names the net of J1.4 (Pin_4)
- net ~{EN2}: no longer names the net of J3.6 (Pin_6)
- no-connect marks 19 -> 21
Other:
- note added: "JST 10pol DIN 8pol Bez. Farbe Vbl. 1 2 (sw) Gnd sw 2 4 (rt) Revox TXD gn 3 3 (ws) Revox RXD ge 4 5 (ge) RS232 +5V 10 1 (br) +5V rt 7 7 (bl) RTS or 8 6 (vio) CTS br"
- note added: "JST 6pol. DIN 6pol. 1 (sw) 1 (gnd) 2 (br) 2 (gnd) 3 (ge) 3 (SerialLink) 4 (bl) 4 (nc) 5 (rt) 5 (+5V) 6 (vio) 6 (nc)"
- note removed: "J1 Revox B203 JST 6pol. DIN 6pol. 1 1 (gnd) 2 2 (gnd) 3 3 (SerialLink) 4 4 (nc) 5 5 (+5V) 6 6 (nc)"
- note removed: "JST 10pol DIN 8pol Bez. Hinweis 1 2 Gnd 2 4 Revox TXD 3 3 Revox RXD 4 5 RS232 +5V 10 1 +5V 7 7 RTS nicht verwendet 8 6 CTS nicht verwendet"
- note removed: "Wichtig, das SerialLink Kabel muss an Port A angeschlossen werden und er Jumper JS1 auf der B203 Hauptplatine muss auf Stellung R gesteckt sein."
