File: Schematic_PCB/RevoxESP32Light/RevoxESP32Light.kicad_sch (KiCad schematic)
At the start: 12 parts, among them J1 SerialLink, J2 Conn_01x04, J3 Conn_01x10, J4 Conn_01x05, J5 Conn_01x04, J6 Conn_01x03, U1 esp32-wemos-d1-mini, U2 TSOP331xx, U3 TTL-RS232 Modul, U6 FXMA108_THT

Commit message: Revox B285 Bugfixing.
Connections:
- net +5V: now also J1.4 (Pin_4); no longer J1.5 (Pin_5)
Other:
- note added: "JST 6pol. DIN 6pol. 1 (sw) 1 (gnd) 2 (br) 2 (gnd) 3 (ge) 3 (SerialLink) 4 (rt) 4 (+5V) 5 (bl) 5 (nc) 6 (vio) 6 (nc)"
- note removed: "JST 6pol. DIN 6pol. 1 (sw) 1 (gnd) 2 (br) 2 (gnd) 3 (ge) 3 (SerialLink) 4 (bl) 4 (nc) 5 (rt) 5 (+5V) 6 (vio) 6 (nc)"
Changed lines of the file:
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@@
 		)
 	)
-	(text "JST 6pol.			DIN 6pol.\n1	(sw)			1 (gnd)\n2	(br)			2 (gnd)\n3	(ge)			3 (SerialLink)\n4	(bl)			4 (nc)\n5	(rt)			5 (+5V)\n6	(vio)			6 (nc)"
+	(text "JST 6pol.			DIN 6pol.\n1	(sw)			1 (gnd)\n2	(br)			2 (gnd)\n3	(ge)			3 (SerialLink)\n4	(rt)			4 (+5V)\n5	(bl)			5 (nc)\n6	(vio)			6 (nc)"
 		(exclude_from_sim no)
 		(at 174.498 51.816 0)
@@
 	)
 	(junction
-		(at 248.92 40.64)
+		(at 55.88 143.51)
 		(diameter 0)
 		(color 0 0 0 0)
 	)
 	(junction
-		(at 55.88 143.51)
+		(at 245.11 124.46)
 		(diameter 0)
 		(color 0 0 0 0)
 	)
 	(junction
-		(at 245.11 124.46)
+		(at 248.92 38.1)
 		(diameter 0)
 		(color 0 0 0 0)
@@
 	)
 	(no_connect
+		(at 257.81 40.64)
+	)
+	(no_connect
 		(at 257.81 43.18)
 	)
@@
 	)
 	(no_connect
-		(at 257.81 38.1)
-	)
-	(no_connect
 		(at 156.21 163.83)
 	)
@@
 	(wire
 		(pts
-			(xy 238.76 40.64) (xy 248.92 40.64)
+			(xy 242.57 38.1) (xy 248.92 38.1)
 		)
 		(stroke
@@
 	(wire
 		(pts
-			(xy 248.92 40.64) (xy 248.92 44.45)
-		)
-		(stroke
-			(width 0)
-			(type default)
-		)
-	)
-	(wire
-		(pts
 			(xy 48.26 124.46) (xy 55.88 124.46)
 		)
@@
 	(wire
 		(pts
+			(xy 248.92 38.1) (xy 248.92 44.45)
+		)
+		(stroke
+			(width 0)
+			(type default)
+		)
+	)
+	(wire
+		(pts
 			(xy 93.98 57.15) (xy 101.6 57.15)
 		)
@@
 	(wire
 		(pts
+			(xy 257.81 38.1) (xy 248.92 38.1)
+		)
+		(stroke
+			(width 0)
+			(type default)
+		)
+	)
+	(wire
+		(pts
 			(xy 53.34 148.59) (xy 58.42 148.59)
 		)
@@
 		)
 	)
-	(wire
-		(pts
-			(xy 248.92 40.64) (xy 257.81 40.64)
-		)
-		(stroke
-			(width 0)
-			(type default)
-		)
-	)
 	(image
 		(at 184.15 30.48)
@@
 	(symbol
 		(lib_id "power:+5V")
-		(at 238.76 40.64 90)
+		(at 242.57 38.1 90)
 		(unit 1)
 		(body_style 1)
@@
 		(fields_autoplaced yes)
 		(property "Reference" "#PWR06"
-			(at 242.57 40.64 0)
+			(at 246.38 38.1 0)
 			(hide yes)
 			(show_name no)
@@
 		)
 		(property "Value" "+5V"
-			(at 234.95 40.6399 90)
+			(at 238.76 38.0999 90)
 			(show_name no)
 			(do_not_autoplace no)
@@
 		)
 		(property "Footprint" ""
-			(at 238.76 40.64 0)
+			(at 242.57 38.1 0)
 			(hide yes)
 			(show_name no)
@@
 		)
 		(property "Datasheet" ""
-			(at 238.76 40.64 0)
+			(at 242.57 38.1 0)
 			(hide yes)
 			(show_name no)
@@
 		)
 		(property "Description" "Power symbol creates a global label with name \"+5V\""
-			(at 238.76 40.64 0)
+			(at 242.57 38.1 0)
 			(hide yes)
 			(show_name no)
