File: Schematic_PCB/RevoxESP32IR/RevoxESP32IR.kicad_pcb (KiCad board)
At the start: 2 copper layers, 120.1 x 73.7 mm, 31 parts, among them J1 SerialLink, J2 Conn_01x04, J3 Conn_01x10, J4 Conn_01x05, J5 Conn_01x04, J6 Conn_01x03, Q1 BC550, Q2 2N2222, Q3 BC550, U1 esp32-wemos-d1-mini, U2 TSOP331xx, U3 TTL-RS232 Modul, U6 FXMA108_THT

Commit message: Anpassung Schematic  und PCB.
Parts:
- R12: value 2,2k -> 1k
Connections:
- J1 pad 4: ~{EN1} -> +5V
- J1 pad 5: +5V -> unconnected-(J1-Pin_5-Pad5)
- J1 pad 6: unconnected-(J1-Pin_6-Pad6) -> ~{EN1}
Routing:
- net ~{EN1}: track 21.7 -> 27.7 mm
Changed lines of the file:
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@@
 			(layers "*.Cu" "*.Mask")
 			(remove_unused_layers no)
-			(net "~{EN1}")
+			(net "+5V")
 			(pinfunction "Pin_4_4")
 			(pintype "passive")
@@
 			(layers "*.Cu" "*.Mask")
 			(remove_unused_layers no)
-			(net "+5V")
+			(net "unconnected-(J1-Pin_5-Pad5)")
 			(pinfunction "Pin_5_5")
-			(pintype "passive")
+			(pintype "passive+no_connect")
 		)
 		(pad "6" thru_hole oval
@@
 			(layers "*.Cu" "*.Mask")
 			(remove_unused_layers no)
-			(net "unconnected-(J1-Pin_6-Pad6)")
+			(net "~{EN1}")
 			(pinfunction "Pin_6_6")
-			(pintype "passive+no_connect")
+			(pintype "passive")
 		)
 		(embedded_fonts no)
@@
 			)
 		)
-		(property "Value" "2,2k"
+		(property "Value" "1k"
 			(at 6.35 2.72 0)
 			(layer "F.Fab")
@@
 	)
 	(segment
-		(start 138.4411 77.6443)
-		(end 134.2609 77.6443)
+		(start 133.5857 78.5043)
+		(end 133.5857 89.2231)
 		(width 0.2)
 		(layer "B.Cu")
@@
 	)
 	(segment
-		(start 134.2609 77.6443)
-		(end 133.5857 78.3195)
+		(start 134.62 76.835)
+		(end 133.59 77.865)
 		(width 0.2)
 		(layer "B.Cu")
@@
 	)
 	(segment
-		(start 133.5857 78.3195)
-		(end 133.5857 89.2231)
+		(start 133.5857 89.2231)
+		(end 130.8608 91.948)
 		(width 0.2)
 		(layer "B.Cu")
@@
 	)
 	(segment
-		(start 139.74 78.9432)
-		(end 138.4411 77.6443)
+		(start 133.59 77.865)
+		(end 133.59 78.5)
 		(width 0.2)
 		(layer "B.Cu")
@@
 	)
 	(segment
-		(start 133.5857 89.2231)
-		(end 130.8608 91.948)
+		(start 144.74 78.9432)
+		(end 142.6318 76.835)
 		(width 0.2)
 		(layer "B.Cu")
@@
 	)
 	(segment
-		(start 202.184 82.884)
-		(end 202.184 96.012)
+		(start 142.6318 76.835)
+		(end 134.62 76.835)
 		(width 0.2)
-		(layer "F.Cu")
-		(net "+5V")
+		(layer "B.Cu")
+		(net "~{EN1}")
 	)
 	(segment
-		(start 155.4837 77.1144)
-		(end 143.8656 77.1144)
+		(start 133.59 78.5)
+		(end 133.5857 78.5043)
+		(width 0.2)
+		(layer "B.Cu")
+		(net "~{EN1}")
+	)
+	(segment
+		(start 202.184 82.884)
+		(end 202.184 96.012)
 		(width 0.2)
 		(layer "F.Cu")
@@
 	)
 	(segment
-		(start 142.24 78.9432)
-		(end 140.4112 80.772)
+		(start 137.9112 80.772)
+		(end 139.74 78.9432)
 		(width 0.2)
 		(layer "F.Cu")
@@
 	)
 	(segment
-		(start 140.4112 80.772)
-		(end 131.4839 80.772)
+		(start 141.5688 77.1144)
+		(end 139.74 78.9432)
 		(width 0.2)
 		(layer "F.Cu")
@@
 	)
 	(segment
-		(start 157.1893 78.82)
-		(end 155.4837 77.1144)
+		(start 131.4839 80.772)
+		(end 137.9112 80.772)
 		(width 0.2)
 		(layer "F.Cu")
@@
 	)
 	(segment
-		(start 142.24 78.74)
-		(end 142.24 78.9432)
+		(start 157.1893 78.82)
+		(end 155.4837 77.1144)
 		(width 0.2)
 		(layer "F.Cu")
@@
 	)
 	(segment
-		(start 131.4839 80.772)
-		(end 130.4679 79.756)
+		(start 155.4837 77.1144)
+		(end 141.5688 77.1144)
 		(width 0.2)
 		(layer "F.Cu")
@@
 	)
 	(segment
-		(start 143.8656 77.1144)
-		(end 142.24 78.74)
+		(start 131.4839 80.772)
+		(end 130.4679 79.756)
 		(width 0.2)
 		(layer "F.Cu")
@@
 		(net "IO04")
 	)
+	(segment
+		(start 142.24 78.74)
+		(end 142.24 78.9432)
+		(width 0.2)
+		(layer "F.Cu")
+		(net "unconnected-(J1-Pin_5-Pad5)")
+	)
 	(zone
